File: pcb/CableChecker.kicad_sch (KiCad schematic)
At the start: 11 parts, among them J1 AudioJack3_SwitchTR, J2 NC3MAAH, J3 NC3FAAH, SW1 RotaryEncoder_Switch_MP, U1 ES8388

Commit message: added adf
Parts:
- added SW2: SW_SP3T, easyeda2kicad:SW-TH_SK13D07VG5, symbol Switch:SW_SP3T
- LED1: renamed from U2; footprint (none) -> LED_SMD:GlowbitL_LED_Strip_1x8
- renumbered U3 to Charger1
Connections:
- net GND: now also SW2.1
- new net SW-1: ESP32_S1. (14), SW2.2
- new net SW-2: ESP32_S1. (14), SW2.3
- new net SW-3: ESP32_S1. (14), SW2.4

Commit message: hardware mostly done
Parts:
- removed C1: 1uF, symbol Device:C
- removed Charger1: ~, Battery:Makerverse USB-C LiPo Charger, symbol Battery_Management:Makerverse_LiPo_Charger
- removed J1: AudioJack3_SwitchTR, symbol Connector_Audio:AudioJack3_SwitchTR
- added CN1: PJ-306M, easyeda2kicad:AUDIO-TH_HOOYA_PJ-306M, symbol easyeda2kicad:PJ-306M
- ESP32_S1: footprint (none) -> RF_Module:ESP32-S3-ZERO
- renumbered U1 to AudioCodec1
Connections:
- net +3.3V: no longer LED1.+ (Vcc)
- net +5V: now also LED1.+ (Vcc)
- net GND: now also AudioCodec1.20 (VMID), CN1.1
- net Ring: now also CN1.2
- net Ring-Shunt: now also CN1.3
- net Tip: now also CN1.4
- net Tip-Shunt: now also CN1.5
