File: pcb/CableChecker.kicad_pcb (KiCad board)
At the start: 2 copper layers, 7 parts, among them J2 NC3MAAH, J3 NC3FAAH, SW1 RotaryEncoder_Switch_MP, U1 ES8388, U2 ESP32-S3

Commit message: added adf
Parts:
- removed U2: ESP32-S3, Package_DFN_QFN:QFN-56-1EP_7x7mm_P0.4mm_EP4x4mm
- added LED1: ~, LED_SMD:GlowbitL_LED_Strip_1x8, B.Cu at (195.6, 110.2)
- added SW2: SW_SP3T, easyeda2kicad:SW-TH_SK13D07VG5, F.Cu at (183.4, 76.0)
- SW1: moved to B.Cu
- moved J2 127.8 mm to (192.4, 131.0), turned to 0 degrees
- moved XFR1 59.5 mm to (196.1, 91.0)
- moved XFR2 58.4 mm to (206.0, 91.0)
- moved U1 51.9 mm to (206.9, 104.5)
- moved J3 50.0 mm to (192.2, 61.8), turned to 90 degrees
- moved SW1 38.4 mm to (203.5, 73.0), turned to 180 degrees
Connections:
- J2 pad 1: unconnected-(J2-Pad1) -> GND
- J2 pad 2: unconnected-(J2-Pad2) -> Net-(J2-Pad2)
- J2 pad 3: unconnected-(J2-Pad3) -> Net-(J2-Pad3)
- J2 pad G: unconnected-(J2-PadG) -> GND
- J3 pad 1: unconnected-(J3-Pad1) -> GND
- J3 pad 2: unconnected-(J3-Pad2) -> Net-(J3-Pad2)
- J3 pad 3: unconnected-(J3-Pad3) -> Net-(J3-Pad3)
- SW1 pad A: unconnected-(SW1-PadA) -> RE-CLK
- SW1 pad B: unconnected-(SW1-PadB) -> RE-DT
- SW1 pad C: unconnected-(SW1-PadC) -> GND
- SW1 pad MP: unconnected-(SW1-PadMP) -> GND
- SW1 pad S1: unconnected-(SW1-PadS1) -> RE-SW
- SW1 pad S2: unconnected-(SW1-PadS2) -> GND
- U1 pad 1: unconnected-(U1-MCLK-Pad1) -> MCLK
- U1 pad 10: unconnected-(U1-VREF-Pad10) -> +3.3V
- U1 pad 12: unconnected-(U1-LOUT1-Pad12) -> LOUT1
- U1 pad 13: unconnected-(U1-HPGND-Pad13) -> GND
- U1 pad 14: unconnected-(U1-ROUT2-Pad14) -> Ring
- U1 pad 15: unconnected-(U1-LOUT2-Pad15) -> Tip
- U1 pad 16: unconnected-(U1-HPVDD-Pad16) -> +3.3V
- U1 pad 17: unconnected-(U1-AVDD-Pad17) -> +3.3V
- U1 pad 18: unconnected-(U1-AGND-Pad18) -> GND
- U1 pad 19: unconnected-(U1-ADCVREF-Pad19) -> +3.3V
- U1 pad 2: unconnected-(U1-DVDD-Pad2) -> +3.3V
- U1 pad 20: unconnected-(U1-VMID-Pad20) -> Net-(U1-VMID)
- U1 pad 24: unconnected-(U1-LIN1-Pad24) -> LIN1
- U1 pad 26: unconnected-(U1-CE-Pad26) -> CE
- U1 pad 27: unconnected-(U1-CDATA-Pad27) -> CDATA
- U1 pad 28: unconnected-(U1-CCLK-Pad28) -> CCLK
- U1 pad 29: unconnected-(U1-EPAD-Pad29) -> GND
- U1 pad 3: unconnected-(U1-PVDD-Pad3) -> +3.3V
- U1 pad 4: unconnected-(U1-DGND-Pad4) -> GND
- U1 pad 5: unconnected-(U1-SCLK-Pad5) -> SCLK
- U1 pad 6: unconnected-(U1-DSDIN-Pad6) -> DSDIN
- U1 pad 7: unconnected-(U1-LRCK-Pad7) -> LRCK
- U1 pad 8: unconnected-(U1-ASDOUT-Pad8) -> ASDOUT
- XFR1 pad 1: unconnected-(XFR1-Pad1) -> Net-(J2-Pad3)
- XFR1 pad 2: unconnected-(XFR1-Pad2) -> LOUT1
- XFR1 pad 5: unconnected-(XFR1-Pad5) -> Net-(J2-Pad2)
- XFR1 pad 6: unconnected-(XFR1-Pad6) -> GND
- XFR2 pad 1: unconnected-(XFR2-Pad1) -> LIN1
- XFR2 pad 2: unconnected-(XFR2-Pad2) -> Net-(J3-Pad3)
- XFR2 pad 5: unconnected-(XFR2-Pad5) -> GND
- XFR2 pad 6: unconnected-(XFR2-Pad6) -> Net-(J3-Pad2)
Other:
- board outline added: 30 x 100 mm

Commit message: hardware mostly done
Parts:
- added CN1: PJ-306M, easyeda2kicad:AUDIO-TH_HOOYA_PJ-306M, F.Cu at (187.0, 121.5)
- added ESP32_S1: ~, RF_Module:ESP32-S3-ZERO, F.Cu at (190.9, 104.2)
- moved SW2 59.0 mm to (183.5, 135.0)
- moved XFR1 33.8 mm to (203.5, 124.0), turned to 90 degrees
- moved AudioCodec1 29.2 mm to (205.8, 75.3), turned to 180 degrees
- moved LED1 20.6 mm to (204.9, 91.8)
- moved XFR2 15.2 mm to (191.1, 88.2), turned to 90 degrees
- moved SW1 4.77 mm to (198.8, 73.4)
- renumbered U1 to AudioCodec1
Connections:
- AudioCodec1 pad 20: Net-(U1-VMID) -> GND
- LED1 pad 1: (no net) -> +5V
- LED1 pad 3: (no net) -> GND
- LED1 pad 4: (no net) -> GND
Routing:
- net GND: track 0.00 -> 167.7 mm, vias 0 -> 2
- net +5V: track 0.00 -> 85.3 mm, vias 0 -> 2
- net LOUT1: track 0.00 -> 64.6 mm
- net Tip: track 0.00 -> 64.3 mm, vias 0 -> 2
- net Ring: track 0.00 -> 59.7 mm, vias 0 -> 2
- net MCLK: track 0.00 -> 56.2 mm, vias 0 -> 1
- net SW-3: track 0.00 -> 49.0 mm
- net CCLK: track 0.00 -> 45.9 mm, vias 0 -> 1
- net SW-2: track 0.00 -> 43.8 mm, vias 0 -> 1
- net CDATA: track 0.00 -> 43.3 mm, vias 0 -> 1
- net SW-1: track 0.00 -> 41.9 mm
- net CE: track 0.00 -> 40.9 mm, vias 0 -> 1
- net ASDOUT: track 0.00 -> 34.8 mm, vias 0 -> 2
- net Net-(J3-Pad2): track 0.00 -> 34.0 mm
- net RE-SW: track 0.00 -> 33.4 mm
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Other:
- board text added: "Joshua Wolfson"

Commit message: finished hardware
Parts:
- moved J3 54.1 mm to (232.2, 98.2), turned to 0 degrees
- moved SW2 51.7 mm to (159.0, 89.5), turned to 180 degrees
- moved J2 43.9 mm to (163.0, 98.4), turned to -90 degrees
- moved AudioCodec1 38.7 mm to (218.7, 111.8), turned to 90 degrees
- moved SW1 38.2 mm to (220.6, 104.8), turned to 90 degrees
- moved XFR1 36.4 mm to (170.0, 109.5), turned to 0 degrees
- moved CN1 32.0 mm to (172.5, 93.0), turned to 0 degrees
- moved LED1 19.3 mm to (202.2, 110.9), turned to 90 degrees
- moved XFR2 17.2 mm to (205.8, 97.1), turned to 0 degrees
- moved ESP32_S1 7.43 mm to (189.8, 96.9), turned to 0 degrees
Other:
- board size 30 x 100 mm -> 100 x 30 mm
